Commit message: feat(driver): add Feetech ros2_control hardware plugin

File: lekiwi_description/urdf/duykhongcay_lekiwi.urdf (robot description, URDF)
Before this commit: robot lekiwi, 16 links, 15 joints
Links:
- link base_footprint: geometry collision mesh filename=package://assets/base_motor_holder_so101_v1.stl; collision mesh filename=package://assets/base_plate_layer1_v5_1__body1.stl
- link gripper: geometry collision mesh filename=package://assets/generic_usb_camera.stl; collision mesh filename=package://assets/sts3215_03a_v1.stl
- link lower_arm: geometry collision mesh filename=package://assets/motor_holder_so101_wrist_v1.stl; collision mesh filename=package://assets/sts3215_03a_v1.stl
- link moving_jaw_so101_v1: geometry collision mesh filename=package://assets/moving_jaw_so101_v1.stl; visual mesh filename=package://assets/moving_jaw_so101_v1.stl
- link omniwheel_7: geometry collision mesh filename=package://assets/duy0cay_omniwheel_mount_for_st3215.stl; collision mesh filename=package://assets/sphere_drive_simplified_hq.stl
- link omniwheel_8: geometry collision mesh filename=package://assets/duy0cay_omniwheel_mount_for_st3215.stl; collision mesh filename=package://assets/sphere_drive_simplified_hq.stl
- link omniwheel_9: geometry collision mesh filename=package://assets/duy0cay_omniwheel_mount_for_st3215.stl; collision mesh filename=package://assets/sphere_drive_simplified_hq.stl
- link rotation_pitch: geometry collision mesh filename=package://assets/base_side_cam_1__body1.stl; collision mesh filename=package://assets/generic_usb_camera.stl
- link upper_arm: geometry collision mesh filename=package://assets/sts3215_03a_v1.stl; collision mesh filename=package://assets/upper_arm_so101_v1.stl
- link wrist: geometry collision mesh filename=package://assets/sts3215_03a_no_horn_v1.stl; collision mesh filename=package://assets/wrist_roll_pitch_so101_v2.stl
Joints:
- removed joint back_wheel
- removed joint elbow_flex
- removed joint gripper
- removed joint left_wheel
- removed joint right_wheel
- removed joint shoulder_lift
- removed joint shoulder_pan
- removed joint wrist_flex
- removed joint wrist_roll
- added joint arm_elbow_flex: type revolute, parent upper_arm, child lower_arm, origin xyz=-0.11257 -0.028 0 rpy=-0 -0 1.57038, axis 0 0 1, limit lower=-1.65765 upper=1.57121 effort=10 velocity=10
- added joint arm_gripper: type revolute, parent gripper, child moving_jaw_so101_v1, origin xyz=0.0202 0.0186 -0.0234 rpy=1.5708 0.000965842 -0, axis 0 0 1, limit lower=-0.0863006 upper=1.65903 effort=10 velocity=10
- added joint arm_shoulder_lift: type revolute, parent rotation_pitch, child upper_arm, origin xyz=-0.0306 -0.0183 -0.0542 rpy=-1.5708 -1.5708 0, axis 0 0 1, limit lower=-1.74533 upper=1.74533 effort=10 velocity=10
- added joint arm_shoulder_pan: type revolute, parent base_footprint, child rotation_pitch, origin xyz=0.0461807 1.27994e-05 0.1696 rpy=3.14159 0 3.13774, axis 0 0 1, limit lower=-1.74919 upper=1.74147 effort=10 velocity=10
- added joint arm_wrist_flex: type revolute, parent lower_arm, child wrist, origin xyz=-0.1349 0.0052 -0 rpy=-0 0 -1.57999, axis 0 0 1, limit lower=-1.56161 upper=1.57999 effort=10 velocity=10
- added joint arm_wrist_roll: type revolute, parent wrist, child gripper, origin xyz=-5.18e-10 -0.0611 0.0181 rpy=1.5708 0.0594906 3.14159, axis 0 0 1, limit lower=-2.64577 upper=2.76475 effort=10 velocity=10
- added joint base_back_wheel: type continuous, parent base_footprint, child omniwheel_8, origin xyz=-0.130267 1.32994e-05 0.065 rpy=-3.14159 -1.5708 0, axis 0 0 1, limit effort=10 velocity=10
- added joint base_left_wheel: type continuous, parent base_footprint, child omniwheel_7, origin xyz=0.0336827 0.0946699 0.065 rpy=1.5708 0 -0.523599, axis 0 0 1, limit effort=10 velocity=10
- added joint base_right_wheel: type continuous, parent base_footprint, child omniwheel_9, origin xyz=0.0336827 -0.0946433 0.065 rpy=-1.5708 0.00357617 0.523599, axis 0 0 1, limit effort=10 velocity=10
- joint gripperframe_frame: origin xyz=-0.0079 -0.000218214 -0.103424 rpy=-1.5708 0 -1.5708 -> xyz=-0.0079 -0.000218214 -0.103424 rpy=-1.5708 -0 -1.5708

Commit message: feat(imu): integrate ICM-20948 IMU sensor and refactor bringup launch scripts
- Implement lekiwi_icm20948_hardware package with ros2_control SensorInterface
- Support Linux i2c-dev communication, AK09916 magnetometer, and gyro auto-calibration
- Export 13 state interfaces (orientation, angular velocity, linear acceleration, magnetic field)
- Update udev rules for I2C bus access and symlink /dev/i2c-imu
- Update CAD-exported URDF with icm20948_imu link/joint and rename xacro_macros.xacro to ros2_control.xacro
- Add lekiwi_imu_broadcaster and lekiwi_magnetometer_broadcaster controllers
- Refactor all bringup launch scripts with declarative argument list comprehensions

File: lekiwi_description/urdf/duykhongcay_lekiwi.urdf (robot description, URDF)
Before this commit: robot lekiwi, 16 links, 15 joints
Links:
- added link icm20948_imu, mass 0
Joints:
- added joint icm20948_imu_frame: type fixed, parent base_footprint, child icm20948_imu, origin xyz=-0.0467018 1.32988e-05 0.412365 rpy=2.35619 -0 1.5708, axis 0 0 0

File: lekiwi_description/urdf/lekiwi_robot.urdf.xacro (robot description, xacro)
@@ -6,12 +6,18 @@
   <xacro:arg name="joint_config_file" default=""/>
   <xacro:arg name="add_transmissions" default="false"/>
+  <xacro:arg name="enable_imu" default="true"/>
+  <xacro:arg name="imu_hardware_type" default="mock"/>
+  <xacro:arg name="imu_i2c_bus" default="1"/>
+  <xacro:arg name="imu_i2c_address" default="0x68"/>
+  <xacro:arg name="imu_auto_calibrate_gyro" default="true"/>
+  <xacro:arg name="imu_gyro_calib_samples" default="500"/>
   <!-- Keep the CAD-generated kinematic model separate from control metadata. -->
   <xacro:include filename="$(find lekiwi_description)/urdf/duykhongcay_lekiwi.urdf"/>
-  <xacro:include filename="$(find lekiwi_description)/urdf/xacro_macros.xacro"/>
+  <xacro:include filename="$(find lekiwi_description)/urdf/ros2_control.xacro"/>
   <xacro:if value="$(arg use_ros2_control)">
-    <xacro:lekiwi_ros2_control
-      hardware_type="$(arg hardware_type)"
-      usb_port="$(arg usb_port)"
-      joint_config_file="$(arg joint_config_file)"/>
+    <xacro:lekiwi_ros2_control hardware_type="$(arg hardware_type)" usb_port="$(arg usb_port)" joint_config_file="$(arg joint_config_file)"/>
+    <xacro:if value="$(arg enable_imu)">
+      <xacro:lekiwi_imu_ros2_control hardware_type="$(arg imu_hardware_type)" i2c_bus="$(arg imu_i2c_bus)" i2c_address="$(arg imu_i2c_address)" auto_calibrate_gyro="$(arg imu_auto_calibrate_gyro)" gyro_calib_samples="$(arg imu_gyro_calib_samples)"/>
+    </xacro:if>
   </xacro:if>
   <xacro:if value="$(arg add_transmissions)">

File: lekiwi_description/urdf/ros2_control.xacro (robot description, xacro)
@@ -46,3 +46,32 @@
     </ros2_control>
   </xacro:macro>
+  <!-- Declares IMU ros2_control sensor component with 13 state interfaces -->
+  <xacro:macro name="lekiwi_imu_ros2_control" params="hardware_type:='mock' i2c_bus:=1 i2c_address:='0x68' auto_calibrate_gyro:='true' gyro_calib_samples:=500">
+    <ros2_control name="LeKiwiImu" type="sensor">
+      <hardware>
+        <plugin>lekiwi_icm20948_hardware/ICM20948SensorHardware</plugin>
+        <param name="mock_sensor">${'true' if hardware_type == 'mock' else 'false'}</param>
+        <param name="i2c_bus">${i2c_bus}</param>
+        <param name="i2c_address">${i2c_address}</param>
+        <param name="auto_calibrate_gyro">${auto_calibrate_gyro}</param>
+        <param name="gyro_calib_samples">${gyro_calib_samples}</param>
+      </hardware>
+      <sensor name="icm20948_imu">
+        <state_interface name="orientation.x"/>
+        <state_interface name="orientation.y"/>
+        <state_interface name="orientation.z"/>
+        <state_interface name="orientation.w"/>
+        <state_interface name="angular_velocity.x"/>
+        <state_interface name="angular_velocity.y"/>
+        <state_interface name="angular_velocity.z"/>
+        <state_interface name="linear_acceleration.x"/>
+        <state_interface name="linear_acceleration.y"/>
+        <state_interface name="linear_acceleration.z"/>
+        <state_interface name="magnetic_field.x"/>
+        <state_interface name="magnetic_field.y"/>
+        <state_interface name="magnetic_field.z"/>
+        <param name="frame_id">icm20948_imu</param>
+      </sensor>
+    </ros2_control>
+  </xacro:macro>
 </robot>

Commit message: fix(description): update robot URDF model and camera frame calibrations

File: lekiwi_description/urdf/duykhongcay_lekiwi.urdf (robot description, URDF)
Before this commit: robot lekiwi, 17 links, 16 joints
Links:
- link base_footprint: mass 0 -> None

Commit message: feat(description): add standalone launch and fix mesh package paths
- Add standalone description.launch.py with fallback support for PC (mock/conda) and Pi (real/xacro)
- Install launch directory in lekiwi_description/CMakeLists.txt
- Fix mesh filename URIs in duykhongcay_lekiwi.urdf to package://lekiwi_description/assets/
- Update AGENTS.md to mandate Mermaid syntax for diagrams

File: lekiwi_description/urdf/duykhongcay_lekiwi.urdf (robot description, URDF)
Before this commit: robot lekiwi, 17 links, 16 joints
Links:
- link base_footprint: geometry collision mesh filename=package://lekiwi_description/assets/base_motor_holder_so101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; collision mesh filename=package://lekiwi_description/assets/base_plate_layer1_v5_1_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
- link gripper: geometry collision mesh filename=package://lekiwi_description/assets/generic_usb_camera.stl; collision mesh filename=package://lekiwi_description/assets/sts3215_03a_v1.stl
- link lower_arm: geometry collision mesh filename=package://lekiwi_description/assets/motor_holder_so101_wris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; collision mesh filename=package://lekiwi_description/assets/sts3215_03a_v1.stl
- link moving_jaw_so101_v1: geometry collision mesh filename=package://lekiwi_description/assets/moving_jaw_so101_v1.stl; visual mesh filename=package://lekiwi_description/assets/moving_jaw_so101_v1.stl
- link omniwheel_7: geometry collision mesh filename=package://lekiwi_description/assets/duy0cay_omniwheel_mount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; collision mesh filename=package://lekiwi_description/assets/sphere_drive_simplified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
- link omniwheel_8: geometry collision mesh filename=package://lekiwi_description/assets/duy0cay_omniwheel_mount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; collision mesh filename=package://lekiwi_description/assets/sphere_drive_simplified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
- link omniwheel_9: geometry collision mesh filename=package://lekiwi_description/assets/duy0cay_omniwheel_mount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; collision mesh filename=package://lekiwi_description/assets/sphere_drive_simplified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
- link rotation_pitch: geometry collision mesh filename=package://lekiwi_description/assets/base_side_cam_1__body1.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; collision mesh filename=package://lekiwi_description/assets/generic_usb_camera.stl
- link upper_arm: geometry collision mesh filename=package://lekiwi_description/assets/sts3215_03a_v1.stl; collision mesh filename=package://lekiwi_description/assets/upper_arm_so101_v1.stl
- link wrist: geometry collision mesh filename=package://lekiwi_description/assets/sts3215_03a_no_horn_v1.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; collision mesh filename=package://lekiwi_description/assets/wrist_roll_pitch_so101_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

Commit message: feat(moveit): add lekiwi_moveit_config package and calibrate joint limits
- Add MoveIt 2 configuration with SRDF planning groups for 5-DoF arm and gripper
- Configure OMPL planning pipelines, kinematics (KDL), and trajectory execution
- Provide demo and standalone RViz launch files for real robot execution
- Relax joint limit bounds in URDF to tolerate physical servo backlash

File: lekiwi_description/urdf/duykhongcay_lekiwi.urdf (robot description, URDF)
Before this commit: robot lekiwi, 17 links, 16 joints
Joints:
- joint arm_elbow_flex: limit lower=-1.65765 upper=1.57121 effort=10 velocity=10 -> lower=-1.75 upper=1.68 effort=10 velocity=10
- joint arm_gripper: limit lower=-0.0863006 upper=1.65903 effort=10 velocity=10 -> lower=-0.15 upper=1.75 effort=10 velocity=10
- joint arm_shoulder_lift: limit lower=-1.74533 upper=1.74533 effort=10 velocity=10 -> lower=-1.85 upper=1.85 effort=10 velocity=10
- joint arm_shoulder_pan: limit lower=-1.74919 upper=1.74147 effort=10 velocity=10 -> lower=-1.85 upper=1.85 effort=10 velocity=10
- joint arm_wrist_flex: limit lower=-1.56161 upper=1.57999 effort=10 velocity=10 -> lower=-1.68 upper=1.68 effort=10 velocity=10
- joint arm_wrist_roll: limit lower=-2.64577 upper=2.76475 effort=10 velocity=10 -> lower=-2.80 upper=2.85 effort=10 velocity=10

Commit message: feat(description): update handeye calibration parameters and clean up URDF camera frames

File: lekiwi_description/urdf/duykhongcay_lekiwi.urdf (robot description, URDF)
Before this commit: robot lekiwi, 17 links, 16 joints
Links:
- removed link stereo_left_optical
- removed link stereo_right_optical
Joints:
- removed joint stereo_left_optical_frame
- removed joint stereo_right_optical_frame

File: lekiwi_description/urdf/sensors_calibration.xacro (robot description, xacro)
@@ -13,6 +13,8 @@
       <xacro:property name="stereo_left_rpy" value="-2.392200 0.013614 -1.566144"/>
     </xacro:unless>
+    <!-- Dummy link for stereo left optical frame -->
+    <link name="stereo_left_optical"/>
     <!-- Calibrated optical frame joint connecting base_footprint to stereo_left_optical -->
-    <joint name="stereo_left_optical_calibrated_joint" type="fixed">
+    <joint name="stereo_left_optical_joint" type="fixed">
       <origin xyz="${stereo_left_xyz}" rpy="${stereo_left_rpy}"/>
       <parent link="base_footprint"/>

Commit message: feat(description): update kinematic base center, joint offsets, and assets
- Align base_footprint to mechanical center of mobile base projection in URDF
- Adjust wheel and arm joint origins to match updated base_footprint frame
- Update stereo left camera hand-eye extrinsics calibration
- Add chess box model assets and updated 3D CAD meshes

File: lekiwi_description/urdf/duykhongcay_lekiwi.urdf (robot description, URDF)
Before this commit: robot lekiwi, 15 links, 14 joints
Links:
- link base_footprint: geometry collision mesh filename=package://lekiwi_description/assets/base_motor_holder_so101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; collision mesh filename=package://lekiwi_description/assets/base_plate_layer1_v5_1_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
Joints:
- joint arm_elbow_flex: limit lower=-1.75 upper=1.68 effort=10 velocity=10 -> lower=-1.65765 upper=1.57121 effort=10 velocity=10
- joint arm_gripper: limit lower=-0.15 upper=1.75 effort=10 velocity=10 -> lower=-0.0863006 upper=1.65903 effort=10 velocity=10
- joint arm_shoulder_lift: limit lower=-1.85 upper=1.85 effort=10 velocity=10 -> lower=-1.74533 upper=1.74533 effort=10 velocity=10
- joint arm_shoulder_pan: limit lower=-1.85 upper=1.85 effort=10 velocity=10 -> lower=-1.74919 upper=1.74147 effort=10 velocity=10; origin xyz=0.0461807 1.27994e-05 0.1696 rpy=3.14159 0 3.13774 -> xyz=0.067148 -5e-07 0.1672 rpy=3.14159 0 3.13774
- joint arm_wrist_flex: limit lower=-1.68 upper=1.68 effort=10 velocity=10 -> lower=-1.56161 upper=1.57999 effort=10 velocity=10
- joint arm_wrist_roll: limit lower=-2.80 upper=2.85 effort=10 velocity=10 -> lower=-2.64577 upper=2.76475 effort=10 velocity=10
- joint base_back_wheel: origin xyz=-0.130267 1.32994e-05 0.065 rpy=-3.14159 -1.5708 0 -> xyz=-0.1093 -0 0.0626 rpy=-3.14159 -1.5708 0
- joint base_left_wheel: origin xyz=0.0336827 0.0946699 0.065 rpy=1.5708 0 -0.523599 -> xyz=0.05465 0.0946566 0.0626 rpy=1.5708 0 -0.523599
- joint base_right_wheel: origin xyz=0.0336827 -0.0946433 0.065 rpy=-1.5708 0.00357617 0.523599 -> xyz=0.05465 -0.0946566 0.0626 rpy=-1.5708 0.00357617 0.523599
- joint baseframe_frame: origin xyz=0.000980687 1.27994e-05 0.1048 rpy=0 -0 0 -> xyz=0.021948 -5e-07 0.1024 rpy=0 0 0
- joint icm20948_imu_frame: origin xyz=-0.0467018 1.32988e-05 0.412365 rpy=2.35619 -0 1.5708 -> xyz=-0.0257345 -6.04e-10 0.409965 rpy=2.35619 -0 1.5708
- joint side_camera_optical_frame: origin xyz=-0.0467438 -0.098278 -0.0699611 rpy=1.0472 -0 -2.44346 -> xyz=-0.0467438 -0.098278 -0.0699611 rpy=1.0472 0 -2.44346

Commit message: feat(description): modularize arm joints xacro and update calibration limits
- Extract arm joint definitions into arm_joints.xacro with dynamic limit binding to DuyKhongCay.json
- Update joint range limits in DuyKhongCay.json
- Rename landmark calibration pose from 'home' to 'approach' across calibration suite

File: lekiwi_description/urdf/duykhongcay_lekiwi.urdf (robot description, URDF)
Before this commit: robot lekiwi, 15 links, 14 joints
Joints:
- removed joint arm_elbow_flex
- removed joint arm_gripper
- removed joint arm_shoulder_lift
- removed joint arm_shoulder_pan
- removed joint arm_wrist_flex
- removed joint arm_wrist_roll

File: lekiwi_description/urdf/lekiwi_robot.urdf.xacro (robot description, xacro)
@@ -24,6 +24,9 @@
   <!-- Include kinematic CAD model and modular subsystems -->
   <xacro:include filename="$(find lekiwi_description)/urdf/duykhongcay_lekiwi.urdf"/>
+  <xacro:include filename="$(find lekiwi_description)/urdf/arm_joints.xacro"/>
   <xacro:include filename="$(find lekiwi_description)/urdf/ros2_control.xacro"/>
   <xacro:include filename="$(find lekiwi_description)/urdf/sensors_calibration.xacro"/>
+  <!-- Instantiate calibrated 6-DOF arm joints from SSOT servo calibration file -->
+  <xacro:lekiwi_arm_joints servo_calib_file="$(arg servo_calib_file)"/>
   <!-- Apply hand-eye extrinsics calibration for stereo left camera -->
   <xacro:stereo_camera_calibration calib_file="$(arg camera_calib_file)"/>

Commit message: refactor(description): remove unused arm_joints xacro and embed joints in URDF
- Remove arm_joints.xacro and embed calibrated arm joints in duykhongcay_lekiwi.urdf
- Update lekiwi_robot.urdf.xacro to reference consolidated URDF model

File: lekiwi_description/urdf/duykhongcay_lekiwi.urdf (robot description, URDF)
Before this commit: robot lekiwi, 15 links, 8 joints
Links:
- link base_footprint: mass None -> 0
Joints:
- added joint arm_elbow_flex: type revolute, parent upper_arm, child lower_arm, origin xyz=-0.11257 -0.028 0 rpy=-0 -0 1.57038, axis 0 0 1, limit lower=-1.65765 upper=1.57121 effort=10 velocity=10
- added joint arm_gripper: type revolute, parent gripper, child moving_jaw_so101_v1, origin xyz=0.0202 0.0186 -0.0234 rpy=1.5708 0.000965842 -0, axis 0 0 1, limit lower=-0.0863006 upper=1.65903 effort=10 velocity=10
- added joint arm_shoulder_lift: type revolute, parent rotation_pitch, child upper_arm, origin xyz=-0.0306 -0.0183 -0.0542 rpy=-1.5708 -1.5708 0, axis 0 0 1, limit lower=-1.74533 upper=1.74533 effort=10 velocity=10
- added joint arm_shoulder_pan: type revolute, parent base_footprint, child rotation_pitch, origin xyz=0.067148 -5e-07 0.1672 rpy=3.14159 0 3.13774, axis 0 0 1, limit lower=-1.74919 upper=1.74147 effort=10 velocity=10
- added joint arm_wrist_flex: type revolute, parent lower_arm, child wrist, origin xyz=-0.1349 0.0052 -0 rpy=-0 0 -1.57999, axis 0 0 1, limit lower=-1.56161 upper=1.57999 effort=10 velocity=10
- added joint arm_wrist_roll: type revolute, parent wrist, child gripper, origin xyz=-5.18e-10 -0.0611 0.0181 rpy=1.5708 0.0594906 3.14159, axis 0 0 1, limit lower=-2.64577 upper=2.76475 effort=10 velocity=10

File: lekiwi_description/urdf/lekiwi_robot.urdf.xacro (robot description, xacro)
@@ -24,9 +24,6 @@
   <!-- Include kinematic CAD model and modular subsystems -->
   <xacro:include filename="$(find lekiwi_description)/urdf/duykhongcay_lekiwi.urdf"/>
-  <xacro:include filename="$(find lekiwi_description)/urdf/arm_joints.xacro"/>
   <xacro:include filename="$(find lekiwi_description)/urdf/ros2_control.xacro"/>
   <xacro:include filename="$(find lekiwi_description)/urdf/sensors_calibration.xacro"/>
-  <!-- Instantiate calibrated 6-DOF arm joints from SSOT servo calibration file -->
-  <xacro:lekiwi_arm_joints servo_calib_file="$(arg servo_calib_file)"/>
   <!-- Apply hand-eye extrinsics calibration for stereo left camera -->
   <xacro:stereo_camera_calibration calib_file="$(arg camera_calib_file)"/>
