Commit message: feat(calibration): support headless hand-eye calibration and register wrist camera extrinsics
- Add headless parameter to HandEyeCalibrationNode to stream compressed HUD telemetry to RViz
- Provide ROS 2 Trigger services for taking samples, computing, saving YAML, and toggling torque
- Align camera subscription QoS to BEST_EFFORT and set valid TF frame fallback
- Configure usb_wrist camera pipeline in gscam for RGB streaming during calibration
- Add wrist_camera_calibration macro in sensors_calibration.xacro and link wrist_camera_optical to gripper

File: lekiwi_description/urdf/duykhongcay_lekiwi.urdf (robot description, URDF)
Before this commit: robot lekiwi, 15 links, 14 joints
Links:
- removed link wrist_camera_optical
- link gripper: geometry collision mesh filename=package://lekiwi_description/assets/body1.stl; collision mesh filename=package://lekiwi_description/assets/generic_usb_camera.stl
Joints:
- removed joint wrist_camera_optical_frame

File: lekiwi_description/urdf/lekiwi_robot.urdf.xacro (robot description, xacro)
@@ -18,6 +18,7 @@
   <xacro:arg name="imu_auto_calibrate_gyro" default="true"/>
   <xacro:arg name="imu_gyro_calib_samples" default="500"/>
-  <!-- Hand-eye camera extrinsics calibration file -->
-  <xacro:arg name="camera_calib_file" default="$(find lekiwi_description)/config/calibration/handeye_calib_stereo_left.yaml"/>
+  <!-- Hand-eye camera extrinsics calibration files -->
+  <xacro:arg name="stereo_left_camera_calib_file" default="$(find lekiwi_description)/config/calibration/handeye_calib_stereo_left.yaml"/>
+  <xacro:arg name="wrist_camera_calib_file" default="$(find lekiwi_description)/config/calibration/handeye_calib_wrist.yaml"/>
   <!-- Feetech STS3215 bus servo calibration file -->
   <xacro:arg name="servo_calib_file" default="$(find lekiwi_description)/config/calibration/DuyKhongCay.json"/>
@@ -27,5 +28,7 @@
   <xacro:include filename="$(find lekiwi_description)/urdf/sensors_calibration.xacro"/>
   <!-- Apply hand-eye extrinsics calibration for stereo left camera -->
-  <xacro:stereo_camera_calibration calib_file="$(arg camera_calib_file)"/>
+  <xacro:stereo_camera_calibration calib_file="$(arg stereo_left_camera_calib_file)"/>
+  <!-- Apply hand-eye extrinsics calibration for wrist camera (Eye-in-Hand) -->
+  <xacro:wrist_camera_calibration calib_file="$(arg wrist_camera_calib_file)"/>
   <!-- Instantiate ros2_control actuators and sensor hardware interfaces -->
   <xacro:if value="$(arg use_ros2_control)">

File: lekiwi_description/urdf/sensors_calibration.xacro (robot description, xacro)
@@ -3,8 +3,8 @@
   LeKiwi Sensor Calibration Transforms
   Loads extrinsic calibration parameters from YAML or falls back to nominal
-  calibrated default offsets to attach stereo optical frames to base_footprint.
+  calibrated default offsets to attach stereo and wrist optical frames.
 -->
 <robot xmlns:xacro="http://www.ros.org/wiki/xacro">
-  <!-- Macro to apply hand-eye extrinsics calibration from YAML or calibrated defaults -->
+  <!-- Macro to apply hand-eye extrinsics calibration from YAML or calibrated defaults for stereo left -->
   <xacro:macro name="stereo_camera_calibration" params="calib_file:=''">
     <xacro:if value="${calib_file != ''}">
@@ -27,3 +27,28 @@
     </joint>
   </xacro:macro>
+  <!-- Macro to apply hand-eye extrinsics calibration from YAML or calibrated defaults for wrist camera (Eye-in-Hand) -->
+  <xacro:macro name="wrist_camera_calibration" params="calib_file:=''">
+    <xacro:if value="${calib_file != ''}">
+      <xacro:property name="wrist_calib_dict" value="${xacro.load_yaml(calib_file)}"/>
+      <xacro:property name="wrist_xyz" value="${wrist_calib_dict['transform']['translation']['x']} ${wrist_calib_dict['transform']['translation']['y']} ${wrist_calib_dict['transform']['translation']['z']}"/>
+      <xacro:property name="wrist_rpy" value="${wrist_calib_dict['metrics']['rotation_rpy_deg'][0] * 3.141592653589793 / 180.0} ${wrist_calib_dict['metrics']['rotation_rpy_deg'][1] * 3.141592653589793 / 180.0} ${wrist_calib_dict['metrics']['rotation_rpy_deg'][2] * 3.141592653589793 / 180.0}"/>
+      <xacro:property name="parent_link" value="${wrist_calib_dict['header']['parent_frame']}"/>
+      <xacro:property name="child_link" value="${wrist_calib_dict['header']['child_frame']}"/>
+    </xacro:if>
+    <xacro:unless value="${calib_file != ''}">
+      <!-- Default calibrated values from Hand-Eye Park solver (2026-10-31) -->
+      <xacro:property name="wrist_xyz" value="-0.012997 0.072954 -0.018753"/>
+      <xacro:property name="wrist_rpy" value="2.473426 0.015952 0.154020"/>
+      <xacro:property name="parent_link" value="gripper"/>
+      <xacro:property name="child_link" value="wrist_camera_optical"/>
+    </xacro:unless>
+    <!-- Dummy link for wrist camera optical frame -->
+    <link name="${child_link}"/>
+    <!-- Calibrated optical frame joint connecting parent (gripper) to wrist_camera_optical -->
+    <joint name="${child_link}_joint" type="fixed">
+      <origin xyz="${wrist_xyz}" rpy="${wrist_rpy}"/>
+      <parent link="${parent_link}"/>
+      <child link="${child_link}"/>
+    </joint>
+  </xacro:macro>
 </robot>
